Commit message: Changed from package:// to (find )

File: fanuc_description/urdf/fanuc.urdf (robot description, URDF)
Before this commit: robot fanuc, 9 links, 8 joints
Links:
- link base_link: geometry collision mesh filename=(find moveit_resources_fanuc_description)/meshes/collision/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; visual mesh filename=(find moveit_resources_fanuc_description)/meshes/visual/bas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
- link link_1: geometry collision mesh filename=(find moveit_resources_fanuc_description)/meshes/collision/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; visual mesh filename=(find moveit_resources_fanuc_description)/meshes/visual/lin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
- link link_2: geometry collision mesh filename=(find moveit_resources_fanuc_description)/meshes/collision/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; visual mesh filename=(find moveit_resources_fanuc_description)/meshes/visual/lin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
- link link_3: geometry collision mesh filename=(find moveit_resources_fanuc_description)/meshes/collision/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; visual mesh filename=(find moveit_resources_fanuc_description)/meshes/visual/lin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
- link link_4: geometry collision mesh filename=(find moveit_resources_fanuc_description)/meshes/collision/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; visual mesh filename=(find moveit_resources_fanuc_description)/meshes/visual/lin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
- link link_5: geometry collision mesh filename=(find moveit_resources_fanuc_description)/meshes/collision/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; visual mesh filename=(find moveit_resources_fanuc_description)/meshes/visual/lin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
- link link_6: geometry collision mesh filename=(find moveit_resources_fanuc_description)/meshes/collision/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; visual mesh filename=(find moveit_resources_fanuc_description)/meshes/visual/lin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

File: panda_description/urdf/panda.urdf (robot description, URDF)
Before this commit: robot panda, 12 links, 11 joints
Links:
- link panda_hand: geometry collision mesh filename=(find moveit_resources_panda_description)/meshes/collision/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; visual mesh filename=(find moveit_resources_panda_description)/meshes/visual/han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
- link panda_leftfinger: geometry collision mesh filename=(find moveit_resources_panda_description)/meshes/collision/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; visual mesh filename=(find moveit_resources_panda_description)/meshes/visual/fin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
- link panda_link0: geometry collision mesh filename=(find moveit_resources_panda_description)/meshes/collision/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; visual mesh filename=(find moveit_resources_panda_description)/meshes/visual/lin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
- link panda_link1: geometry collision mesh filename=(find moveit_resources_panda_description)/meshes/collision/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; visual mesh filename=(find moveit_resources_panda_description)/meshes/visual/lin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
- link panda_link2: geometry collision mesh filename=(find moveit_resources_panda_description)/meshes/collision/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; visual mesh filename=(find moveit_resources_panda_description)/meshes/visual/lin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
- link panda_link3: geometry collision mesh filename=(find moveit_resources_panda_description)/meshes/collision/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; visual mesh filename=(find moveit_resources_panda_description)/meshes/visual/lin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
- link panda_link4: geometry collision mesh filename=(find moveit_resources_panda_description)/meshes/collision/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; visual mesh filename=(find moveit_resources_panda_description)/meshes/visual/lin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
- link panda_link5: geometry collision mesh filename=(find moveit_resources_panda_description)/meshes/collision/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; visual mesh filename=(find moveit_resources_panda_description)/meshes/visual/lin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
- link panda_link6: geometry collision mesh filename=(find moveit_resources_panda_description)/meshes/collision/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; visual mesh filename=(find moveit_resources_panda_description)/meshes/visual/lin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
- link panda_link7: geometry collision mesh filename=(find moveit_resources_panda_description)/meshes/collision/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; visual mesh filename=(find moveit_resources_panda_description)/meshes/visual/lin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
- link panda_rightfinger: geometry collision mesh filename=(find moveit_resources_panda_description)/meshes/collision/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; visual mesh filename=(find moveit_resources_panda_description)/meshes/visual/fin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
